File: Interface.kicad_sch (KiCad schematic)
At the start: 19 parts, among them J1 IDC 2x10p 夹板, J2 USB_C_Receptacle_USB2.0, Q1 AO3401A, Q2 2N7002, Q3 AO3401A, Q4 2N7002, U14 MT9700, U15 ESD0524P, U16 ESD0524P, U17 ESD0524P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

Commit message: update: 更新设计
Parts:
- J2: footprint My USB Connector:USB-C-SMD_SHOU_TYPE-C-16P-CB1.6 -> My USB Connector:USB-C-SMD_CX90M-16P
Changed lines of the file:
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@@
 			)
 		)
-		(property "Footprint" "My USB Connector:USB-C-SMD_SHOU_TYPE-C-16P-CB1.6"
+		(property "Footprint" "My USB Connector:USB-C-SMD_CX90M-16P"
 			(at 31.75 38.1 0)
 			(effects
