File: Power.kicad_sch (KiCad schematic)
At the start: 44 parts, among them U1 HPM5301IEG1, U10 EA3036C, U13 LMV321

Commit message: update: 更新设计
Parts:
- C52: value 1.3n -> 1n
- C54: value 910p -> 1n
- C7, C8: footprint Capacitor_SMD:C_0603_1608Metric -> Capacitor_SMD:C_0402_1005Metric
Changed lines of the file:
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@@
 			)
 		)
-		(property "Value" "1.3n"
+		(property "Value" "1n"
 			(at 192.278 100.584 90)
 			(effects
@@
 			)
 		)
-		(property "Value" "910p"
+		(property "Value" "1n"
 			(at 173.736 122.936 0)
 			(effects
@@
 			)
 		)
-		(property "Footprint" "Capacitor_SMD:C_0603_1608Metric"
+		(property "Footprint" "Capacitor_SMD:C_0402_1005Metric"
 			(at 18.7452 54.61 0)
 			(effects
@@
 			)
 		)
-		(property "Footprint" "Capacitor_SMD:C_0603_1608Metric"
+		(property "Footprint" "Capacitor_SMD:C_0402_1005Metric"
 			(at 23.8252 54.61 0)
 			(effects

Commit message: update: 1.1.0设计
Parts:
- added unit 3 of U10
- added unit 2 of U10
Connections:
- net +5V: now also U10.7 (VIN2), U10.8 (EN2); no longer U10.7 (VIN2), U10.8 (EN2)
- net GND: now also C51.2, U10.1 (GND3), U10.18 (EN3), U10.4 (GND2), U10.5 (GND2); no longer C51.1, U10.18 (EN3), U10.4 (GND2), U10.5 (GND2)
- net TRANS_FB: now also U10.3 (FB2); no longer U10.3 (FB2)
- net TRANS_VCC: now also C51.1; no longer C51.2
- net at L3.2: now also U10.6 (LX2); no longer U10.6 (LX2)
- no-connect marks 4 -> 3
Other:
- moved on the sheet: C40, C41, C46, C47, C48, C49, L2, R2, R3
