File: HSLinkPro.kicad_pcb (KiCad board)
At the start: 4 copper layers, 26 x 35 mm, 109 parts, among them J1 IDC 2x10p 夹板, J2 USB_C_Receptacle_USB2.0, J3 Header, Q1 AO3401A, Q2 2N7002, Q3 AO3401A, Q4 2N7002, U1 HPM5301IEG1, U10 EA3036C, U11 SN74LVC1T45DCK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

Commit message: update: 添加一些丝印
Other:
- board text added: "+5V"
- board text added: "DTR"
- board text added: "GND"
- board text added: "NC"
- board text added: "RTS"
- board text added: "RX"
- board text added: "SRST"
- board text added: "TCK"
- board text added: "TDI"
- board text added: "TDO"
- board text added: "TMS"
- board text added: "TRST"
- board text added: "TV_{CC}"
- board text added: "TX"
- board text added: "V_{REF}"

Commit message: update: 更新设计
Parts:
- removed J3: Header, Connector_PinHeader_1.27mm:PinHeader_1x02_P1.27mm_Vertical
- added G*** (x2): LOGO, LOGO, F.Cu at (113.7, 35.4)
- added G***: LOGO, LOGO, F.Cu at (135.4, 36.4)
- added G***: LOGO, LOGO, F.Cu at (123.8, 38.9)
- added SW1: 1TS028A-1900-0600-CT, My Switch:SW-SMD_4P-L2.8-W1.9-P1.20-LS3.0_1TS028A, F.Cu at (106.8, 52.5)
- C7, C8: footprint Capacitor_SMD:C_0603_1608Metric -> Capacitor_SMD:C_0402_1005Metric
- J2: footprint My USB Connector:USB-C-SMD_SHOU_TYPE-C-16P-CB1.6 -> My USB Connector:USB-C-SMD_CX90M-16P
- moved R17 1.54 mm to (109.2, 52.3), turned to -90 degrees
- moved R18 1.52 mm to (104.4, 52.3), turned to -90 degrees
- moved C8 0.66 mm to (112.0, 51.4)
- moved C7 0.65 mm to (111.1, 51.4)
- moved J2 0.30 mm to (96.9, 44.5)
- turned C57 to 180 degrees
- turned D1 to -90 degrees
Connections:
- U1 pad 1: /UART_DTR -> unconnected-(U1B-PA04/URT1.CTS/SPI0.CS0/TRGM0.P04/JTAG.TDO-Pad1)
- U1 pad 38: unconnected-(U1B-PA30/SPI1.DAT2/XPI0.CA_D1/TRGM0.P06/USB0.PWR-Pad38) -> /SWDIO_DIR
- U1 pad 40: /SWDIO_DIR -> /SWDIO/TMS
- U1 pad 46: unconnected-(U1B-PA07/TMR0.COMP0/URT1.TXD/I2C1.SCL/SPI0.MOSI/TRGM0.P07/JTAG.TMS-Pad46) -> /UART_RTS
- U1 pad 47: unconnected-(U1B-PA06/TMR0.CAPT0/URT1.RXD/I2C1.SDA/SPI0.MISO/TRGM0.P06/JTAG.TCK-Pad47) -> /UART_DTR
- U1 pad 48: /UART_RTS -> unconnected-(U1B-PA05/TMR1.COMP2/URT1.DE/URT1.RTS/SPI0.SCLK/TRGM0.P05/JTAG.TDI-Pad48)
Routing:
- net +3V3: track 145.1 -> 152.4 mm, vias 17 -> 18
- net VBUS: track 20.5 -> 27.8 mm, vias 3 -> 4
- net VDD_SOC: track 48.6 -> 44.8 mm
- net /USB_D+: track 6.05 -> 9.00 mm, vias 0 -> 2
- net /BOOT1: track 7.03 -> 9.77 mm, vias 1 -> 2
- net TRANS_VCC: track 38.2 -> 40.7 mm
- net /BOOT0: track 16.7 -> 19.1 mm
- net /USB_D-: track 5.60 -> 7.79 mm, vias 0 -> 2
- net /UART_DTR: track 9.73 -> 11.8 mm
- net /UART_RTS: track 12.7 -> 14.2 mm
- net /VREF: track 7.78 -> 8.89 mm
- net Net-(J2-CC2): track 3.95 -> 4.91 mm
- net /SWDIO_DIR: track 12.2 -> 11.3 mm
- net GND: track 54.1 -> 53.2 mm, vias 57 -> 54
- net Net-(J2-CC1): track 1.52 -> 2.37 mm
Other:
- outline, holes or cut-outs redrawn
- board text added: "V1.1.0"
- board text removed: "V1.0.0"

Commit message: update: 1.1.0设计
Parts:
- added J3: Header 1.27 4P, Connector_PinHeader_1.27mm:PinHeader_1x04_P1.27mm_Vertical, F.Cu at (97.2, 57.5)
- added R22: 22R, Resistor_SMD:R_0402_1005Metric, F.Cu at (101.6, 42.9)
- added R23: 22R, Resistor_SMD:R_0402_1005Metric, F.Cu at (101.6, 41.9)
- C52: value 1.3n -> 1n
- C54: value 910p -> 1n
- moved R14 9.06 mm to (94.4, 37.5), turned to 180 degrees
- moved C7 0.63 mm to (110.6, 51.0), turned to 180 degrees
- moved C8 0.61 mm to (112.4, 50.9), turned to 0 degrees
- turned C51 to 180 degrees
Connections:
- C51 pad 1: GND -> TRANS_VCC
- C51 pad 2: TRANS_VCC -> GND
- U1 pad 11: /UART_RX -> /ISP_RX
- U1 pad 12: /UART_TX -> /ISP_TX
- U1 pad 2: unconnected-(U1B-PA08/TMR0.COMP1/URT2.TXD/I2C2.SCL/SPI3.CS2/JTAG.TRST-Pad2) -> /UART_TX
- U1 pad 3: unconnected-(U1B-PA09/TMR0.CAPT1/URT2.RXD/I2C2.SDA/SPI3.CS1-Pad3) -> /UART_RX
- U1 pad 39: /SWDIO/TMS -> Net-(U1B-PA29/I2C3.SCL/SPI1.MOSI/XPI0.CA_D2/TRGM0.P05/USB0.OC)
- U1 pad 40: /SWDIO/TMS -> Net-(U1B-PA28/I2C3.SDA/SPI1.MISO/XPI0.CA_D0/TRGM0.P04)
- U10 pad 1: unconnected-(U10-GND3-Pad1) -> GND
Routing:
- net /ISP_RX: track 0.00 -> 23.0 mm, vias 0 -> 2
- net /ISP_TX: track 0.00 -> 22.9 mm, vias 0 -> 2
- net GND: track 53.2 -> 64.4 mm, vias 54 -> 62
- net Net-(J2-CC1): track 2.37 -> 10.8 mm, vias 0 -> 2
- net +5V: track 100.3 -> 97.1 mm, vias 9 -> 10
- net +3V3: track 152.4 -> 155.5 mm
- net /UART_TX: track 10.1 -> 13.0 mm
- net VDD_SOC: track 44.8 -> 47.5 mm
- net /UART_RX: track 12.5 -> 14.9 mm
- net VBUS: track 27.8 -> 25.5 mm, vias 4 -> 6
- net /Power/TRANS_VREF: track 26.4 -> 28.3 mm
- net Net-(U1B-PA29/I2C3.SCL/SPI1.MOSI/XPI0.CA_D2/TRGM0.P05/USB0.OC): track 0.00 -> 1.53 mm
- net Net-(U1B-PA28/I2C3.SDA/SPI1.MISO/XPI0.CA_D0/TRGM0.P04): track 0.00 -> 1.35 mm
- net TRANS_VCC_OUT: track 5.27 -> 4.51 mm
- net /TRANS_PWM: track 12.3 -> 11.5 mm
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Other:
- board text added: "BOOT"
- board text added: "G"
- board text added: "R"
- board text added: "T"
- board text added: "V"
- board text removed: "V1.1.0"

Commit message: update: 更新设计
Parts:
- added R24: 22R, Resistor_SMD:R_0402_1005Metric, F.Cu at (114.8, 41.9)
- added R25: 22R, Resistor_SMD:R_0402_1005Metric, F.Cu at (113.8, 41.9)
- added R26: 22R, Resistor_SMD:R_0402_1005Metric, F.Cu at (114.8, 48.1)
- added R27: 22R, Resistor_SMD:R_0402_1005Metric, F.Cu at (113.8, 37.3)
- added R28: 100R, Resistor_SMD:R_0402_1005Metric, F.Cu at (114.8, 37.3)
- added R29: 100R, Resistor_SMD:R_0402_1005Metric, F.Cu at (113.8, 48.1)
- added R30: 100R, Resistor_SMD:R_0402_1005Metric, F.Cu at (113.8, 56.3)
- added R31: 100R, Resistor_SMD:R_0402_1005Metric, F.Cu at (114.8, 56.3)
- added R32: 100R, Resistor_SMD:R_0402_1005Metric, F.Cu at (114.3, 52.2)
- added R33: 100R, Resistor_SMD:R_0402_1005Metric, F.Cu at (112.9, 52.6)
- moved U18 0.98 mm to (114.3, 54.1)
- moved G*** 0.54 mm to (113.2, 35.4) (x2)
Connections:
- U1 pad 19: /P_EN -> unconnected-(U1B-PY00/URT0.TXD/USB0.ID/PMIC_PY00/PURT.TXD/PTMR.COMP0/SOC.GPIO_Y00-Pad19)
- U1 pad 37: unconnected-(U1B-PA31/SPI1.DAT3/XPI0.CA_CS0/TRGM0.P07/USB0.ID-Pad37) -> /P_EN
- U11 pad 4: /Interface /UART_DTR -> Net-(U11-B)
- U12 pad 4: /Interface /UART_RTS -> Net-(U12-B)
- U2 pad 4: /Interface /SWCLK/TCK -> Net-(U2-B)
- U3 pad 4: /Interface /SWDIO/TMS -> Net-(U3-B)
- U4 pad 4: /Interface /TDO -> Net-(U4-B)
- U5 pad 4: /Interface /<NO NET> -> Net-(U5-B)
- U6 pad 4: /Interface /TRST -> Net-(U6-B)
- U7 pad 4: /Interface /SRST -> Net-(U7-B)
- U8 pad 4: /Interface /UART_TX -> Net-(U8-B)
- U9 pad 4: /Interface /UART_RX -> Net-(U9-B)
Routing:
- net Net-(U4-B): track 0.00 -> 18.9 mm, vias 0 -> 2
- net /Interface /TDO: track 22.2 -> 3.40 mm, vias 2 -> 0
- net Net-(U3-B): track 0.00 -> 16.3 mm, vias 0 -> 2
- net Net-(U7-B): track 0.00 -> 14.7 mm, vias 0 -> 2
- net /Interface /TRST: track 20.0 -> 5.35 mm, vias 2 -> 0
- net /Interface /SRST: track 18.7 -> 4.43 mm, vias 2 -> 0
- net /Interface /SWDIO/TMS: track 17.9 -> 3.81 mm, vias 2 -> 0
- net Net-(U6-B): track 0.00 -> 13.9 mm, vias 0 -> 2
- net Net-(U2-B): track 0.00 -> 12.2 mm, vias 0 -> 2
- net Net-(U11-B): track 0.00 -> 11.5 mm, vias 0 -> 2
- net Net-(U12-B): track 0.00 -> 11.5 mm, vias 0 -> 2
- net /Interface /UART_RTS: track 16.1 -> 6.24 mm, vias 3 -> 1
- net /Interface /<NO NET>: track 14.0 -> 4.47 mm, vias 2 -> 0
- net /Interface /UART_DTR: track 17.0 -> 7.88 mm, vias 3 -> 1
- net /P_EN: track 39.5 -> 47.8 mm, vias 5 -> 6
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Other:
- board text added: "BL"
- board text removed: "BOOT"
