File: HSLinkPro.kicad_sch (KiCad schematic)
At the start: 16 parts, among them J3 Header, U1 HPM5301IEG1, Y1 24M

Commit message: update: 更新设计
Parts:
- removed J3: Header, Connector_PinHeader_1.27mm:PinHeader_1x02_P1.27mm_Vertical, symbol Connector_Generic:Conn_01x02
- added SW1: 1TS028A-1900-0600-CT, My Switch:SW-SMD_4P-L2.8-W1.9-P1.20-LS3.0_1TS028A, symbol Switch:SW_Push
Connections:
- net +3V3: now also SW1.2
- net BOOT1: now also SW1.1
- net SWDIO/TMS: now also U1.40 (PA28/I2C3.SDA/SPI1.MISO/XPI0.CA_D0/TRGM0.P04)
- net SWDIO_DIR: now also U1.38 (PA30/SPI1.DAT2/XPI0.CA_D1/TRGM0.P06/USB0.PWR); no longer U1.40 (PA28/I2C3.SDA/SPI1.MISO/XPI0.CA_D0/TRGM0.P04)
- net UART_DTR: now also U1.47 (PA06/TMR0.CAPT0/URT1.RXD/I2C1.SDA/SPI0.MISO/TRGM0.P06/JTAG.TCK); no longer U1.1 (PA04/URT1.CTS/SPI0.CS0/TRGM0.P04/JTAG.TDO)
- net UART_RTS: now also U1.46 (PA07/TMR0.COMP0/URT1.TXD/I2C1.SCL/SPI0.MOSI/TRGM0.P07/JTAG.TMS); no longer U1.48 (PA05/TMR1.COMP2/URT1.DE/URT1.RTS/SPI0.SCLK/TRGM0.P05/JTAG.TDI)
- no-connect marks 9 -> 8
Changed lines of the file:
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@@
 	)
 	(no_connect
-		(at 30.48 41.91)
-	)
-	(no_connect
 		(at 30.48 46.99)
 	)
@@
 	)
 	(no_connect
-		(at 30.48 115.57)
+		(at 30.48 34.29)
 	)
 	(no_connect
-		(at 30.48 39.37)
+		(at 30.48 115.57)
 	)
 	(no_connect
-		(at 30.48 67.31)
+		(at 30.48 36.83)
 	)
 	(wire
@@
 	(wire
 		(pts
+			(xy 19.05 41.91) (xy 30.48 41.91)
+		)
+		(stroke
+			(width 0)
+			(type default)
+		)
+	)
+	(wire
+		(pts
 			(xy 82.55 132.08) (xy 82.55 134.62)
 		)
@@
 	(wire
 		(pts
+			(xy 19.05 67.31) (xy 30.48 67.31)
+		)
+		(stroke
+			(width 0)
+			(type default)
+		)
+	)
+	(wire
+		(pts
 			(xy 19.05 105.41) (xy 30.48 105.41)
 		)
@@
 	(wire
 		(pts
-			(xy 180.34 22.86) (xy 193.04 22.86)
+			(xy 57.15 147.32) (xy 63.5 147.32)
 		)
 		(stroke
@@
 	(wire
 		(pts
-			(xy 19.05 107.95) (xy 30.48 107.95)
-		)
-		(stroke
-			(width 0)
-			(type default)
-		)
-	)
-	(wire
-		(pts
-			(xy 19.05 34.29) (xy 30.48 34.29)
+			(xy 180.34 22.86) (xy 193.04 22.86)
 		)
 		(stroke
@@
 	(wire
 		(pts
-			(xy 19.05 36.83) (xy 30.48 36.83)
+			(xy 19.05 107.95) (xy 30.48 107.95)
 		)
 		(stroke
@@
 	(wire
 		(pts
-			(xy 73.66 147.32) (xy 74.93 147.32)
-		)
-		(stroke
-			(width 0)
-			(type default)
-		)
-	)
-	(wire
-		(pts
 			(xy 134.62 129.54) (xy 134.62 130.81)
 		)
@@
 	(wire
 		(pts
-			(xy 134.62 138.43) (xy 134.62 139.7)
+			(xy 83.82 147.32) (xy 73.66 147.32)
 		)
 		(stroke
@@
 	(wire
 		(pts
-			(xy 82.55 146.05) (xy 82.55 149.86)
+			(xy 134.62 138.43) (xy 134.62 139.7)
 		)
 		(stroke
@@
 	(wire
 		(pts
-			(xy 73.66 149.86) (xy 82.55 149.86)
-		)
-		(stroke
-			(width 0)
-			(type default)
-		)
-	)
-	(wire
-		(pts
 			(xy 19.05 49.53) (xy 30.48 49.53)
 		)
@@
 	(wire
 		(pts
+			(xy 83.82 144.78) (xy 83.82 147.32)
+		)
+		(stroke
+			(width 0)
+			(type default)
+		)
+	)
+	(wire
+		(pts
 			(xy 19.05 54.61) (xy 30.48 54.61)
 		)
@@
 	(wire
 		(pts
+			(xy 19.05 39.37) (xy 30.48 39.37)
+		)
+		(stroke
+			(width 0)
+			(type default)
+		)
+	)
+	(wire
+		(pts
 			(xy 13.97 127) (xy 13.97 144.78)
 		)
@@
 	)
 	(label "UART_DTR"
-		(at 19.05 34.29 0)
+		(at 180.34 43.18 0)
 		(fields_autoplaced yes)
 		(effects
@@
 		)
 	)
-	(label "UART_DTR"
-		(at 180.34 43.18 0)
+	(label "UART_TX"
+		(at 19.05 24.13 0)
 		(fields_autoplaced yes)
 		(effects
@@
 		)
 	)
-	(label "UART_TX"
-		(at 19.05 24.13 0)
+	(label "SWDIO/TMS"
+		(at 19.05 62.23 0)
 		(fields_autoplaced yes)
 		(effects
@@
 	)
 	(label "UART_RTS"
+		(at 19.05 41.91 0)
+		(fields_autoplaced yes)
+		(effects
+			(font
+				(size 1.27 1.27)
+			)
+			(justify left bottom)
+		)
+	)
+	(label "UART_RTS"
 		(at 180.34 45.72 0)
 		(fields_autoplaced yes)
@@
 		)
 	)
+	(label "SWDIO_DIR"
+		(at 19.05 67.31 0)
+		(fields_autoplaced yes)
+		(effects
+			(font
+				(size 1.27 1.27)
+			)
+			(justify left bottom)
+		)
+	)
 	(label "XIN"
 		(at 19.05 133.35 0)
@@
 	)
 	(label "BOOT1"
-		(at 74.93 147.32 0)
+		(at 57.15 147.32 0)
 		(fields_autoplaced yes)
 		(effects
@@
 		)
 	)
-	(label "SWDIO_DIR"
-		(at 19.05 62.23 0)
-		(fields_autoplaced yes)
-		(effects
-			(font
-				(size 1.27 1.27)
-			)
-			(justify left bottom)
-		)
-	)
 	(label "TDO"
 		(at 180.34 30.48 0)
@@
 		)
 	)
-	(label "UART_RX"
-		(at 180.34 50.8 0)
+	(label "UART_DTR"
+		(at 19.05 39.37 0)
 		(fields_autoplaced yes)
 		(effects
@@
 		)
 	)
-	(label "BOOT1"
-		(at 19.05 31.75 0)
+	(label "UART_RX"
+		(at 180.34 50.8 0)
 		(fields_autoplaced yes)
 		(effects
@@
 		)
 	)
-	(label "ADC_VREF"
-		(at 19.05 74.93 0)
+	(label "BOOT1"
+		(at 19.05 31.75 0)
 		(fields_autoplaced yes)
 		(effects
@@
 		)
 	)
-	(label "UART_RTS"
-		(at 19.05 36.83 0)
+	(label "ADC_VREF"
+		(at 19.05 74.93 0)
 		(fields_autoplaced yes)
 		(effects
@@
 	(symbol
 		(lib_id "power:+3V3")
-		(at 82.55 146.05 0)
+		(at 83.82 144.78 0)
 		(unit 1)
 		(exclude_from_sim no)
@@
 		(dnp no)
 		(property "Reference" "#PWR0108"
-			(at 82.55 149.86 0)
+			(at 83.82 148.59 0)
 			(effects
 				(font
@@
 		)
 		(property "Value" "+3V3"
-			(at 82.55 142.494 0)
+			(at 83.82 141.224 0)
 			(effects
 				(font
@@
 		)
 		(property "Footprint" ""
-			(at 82.55 146.05 0)
+			(at 83.82 144.78 0)
 			(effects
 				(font
@@
 		)
 		(property "Datasheet" ""
-			(at 82.55 146.05 0)
+			(at 83.82 144.78 0)
 			(effects
 				(font
@@
 		)
 		(property "Description" "Power symbol creates a global label with name \"+3V3\""
-			(at 82.55 146.05 0)
+			(at 83.82 144.78 0)
 			(effects
 				(font
@@
 	)
 	(symbol
-		(lib_id "Connector_Generic:Conn_01x02")
-		(at 68.58 147.32 0)
-		(mirror y)
-		(unit 1)
-		(exclude_from_sim yes)
-		(in_bom no)
-		(on_board yes)
-		(dnp yes)
-		(fields_autoplaced yes)
-		(property "Reference" "J3"
-			(at 68.58 140.97 0)
-			(effects
-				(font
-					(size 1.27 1.27)
-				)
-			)
-		)
-		(property "Value" "Header"
-			(at 68.58 143.51 0)
-			(effects
-				(font
-					(size 1.27 1.27)
-				)
-			)
-		)
-		(property "Footprint" "Connector_PinHeader_1.27mm:PinHeader_1x02_P1.27mm_Vertical"
-			(at 68.58 147.32 0)
-			(effects
-				(font
-					(size 1.27 1.27)
-				)
-				(hide yes)
-			)
-		)
-		(property "Datasheet" "~"
-			(at 68.58 147.32 0)
-			(effects
-				(font
-					(size 1.27 1.27)
-				)
-				(hide yes)
-			)
-		)
-		(property "Description" "Generic connector, single row, 01x02, script generated (kicad-library-utils/schlib/autogen/connector/)"
-			(at 68.58 147.32 0)
-			(effects
-				(font
-					(size 1.27 1.27)
-				)
-				(hide yes)
-			)
-		)
-		(pin "2"
-		)
-		(pin "1"
-		)
-		(instances
-			(project ""
-				(path "/5e2c1440-f6a4-4887-af75-aa6afc882006"
-					(reference "J3")
-					(unit 1)
-				)
-			)
-		)
-	)
-	(symbol
 		(lib_id "HPM5300_Library:HPM5301IEG1")
 		(at 88.9 67.31 0)
@@
 					(unit 1)
 				)
+			)
+		)
+	)
+	(symbol
+		(lib_id "Switch:SW_Push")
+		(at 68.58 147.32 0)
+		(unit 1)
+		(exclude_from_sim no)
+		(in_bom yes)
+		(on_board yes)
+		(dnp no)
+		(fields_autoplaced yes)
+		(property "Reference" "SW1"
+			(at 68.58 139.7 0)
+			(effects
+				(font
+					(size 1.27 1.27)
+				)
+			)
+		)
+		(property "Value" "1TS028A-1900-0600-CT"
+			(at 68.58 142.24 0)
+			(effects
+				(font
+					(size 1.27 1.27)
+				)
+			)
+		)
+		(property "Footprint" "My Switch:SW-SMD_4P-L2.8-W1.9-P1.20-LS3.0_1TS028A"
+			(at 68.58 142.24 0)
+			(effects
+				(font
+					(size 1.27 1.27)
+				)
+				(hide yes)
+			)
+		)
+		(property "Datasheet" "~"
+			(at 68.58 142.24 0)
+			(effects
+				(font
+					(size 1.27 1.27)
+				)
+				(hide yes)
+			)
+		)
+		(property "Description" "Push button switch, generic, two pins"
+			(at 68.58 147.32 0)
+			(effects
+				(font
+					(size 1.27 1.27)
+				)
+				(hide yes)
+			)
+		)
+		(pin "1"
+		)
+		(pin "2"
+		)
+		(instances
+			(project ""
+				(path "/5e2c1440-f6a4-4887-af75-aa6afc882006"
+					(reference "SW1")
+					(unit 1)
+				)

Commit message: update: 1.1.0设计
Parts:
- added J3: Header 1.27 4P, Connector_PinHeader_1.27mm:PinHeader_1x04_P1.27mm_Vertical, symbol Connector_Generic:Conn_01x04
- added R22, R23: 22R, Resistor_SMD:R_0402_1005Metric, symbol Device:R
Connections:
- net +3V3: now also J3.1 (Pin_1)
- net GND: now also J3.4 (Pin_4)
- net SWDIO/TMS: now also R22.1, R23.1; no longer U1.39 (PA29/I2C3.SCL/SPI1.MOSI/XPI0.CA_D2/TRGM0.P05/USB0.OC), U1.40 (PA28/I2C3.SDA/SPI1.MISO/XPI0.CA_D0/TRGM0.P04)
- net UART_RX: now also U1.3 (PA09/TMR0.CAPT1/URT2.RXD/I2C2.SDA/SPI3.CS1); no longer U1.11 (PA01/TMR1.CAPT0/URT0.RXD/TRGM0.P01/ACMP.COMP0)
- net UART_TX: now also U1.2 (PA08/TMR0.COMP1/URT2.TXD/I2C2.SCL/SPI3.CS2/JTAG.TRST); no longer U1.12 (PA00/TMR1.COMP0/URT0.TXD/TRGM0.P00)
- new net: R23.2, U1.39 (PA29/I2C3.SCL/SPI1.MOSI/XPI0.CA_D2/TRGM0.P05/USB0.OC)
- new net: R22.2, U1.40 (PA28/I2C3.SDA/SPI1.MISO/XPI0.CA_D0/TRGM0.P04)
- new net ISP_RX: J3.3 (Pin_3), U1.11 (PA01/TMR1.CAPT0/URT0.RXD/TRGM0.P01/ACMP.COMP0)
- new net ISP_TX: J3.2 (Pin_2), U1.12 (PA00/TMR1.COMP0/URT0.TXD/TRGM0.P00)
- no-connect marks 8 -> 6
Other:
- moved on the sheet: C21, C22, C23, C57, D1, R1, R10, R11, R12, R17, R18, R21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

Commit message: update: 更新设计
Connections:
- net P_EN: now also U1.37 (PA31/SPI1.DAT3/XPI0.CA_CS0/TRGM0.P07/USB0.ID); no longer U1.19 (PY00/URT0.TXD/USB0.ID/PMIC_PY00/PURT.TXD/PTMR.COMP0/SOC.GPIO_Y00)
Changed lines of the file:
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@@
-	)
-	(no_connect
-		(at 34.29 69.85)
 	)
 	(no_connect
@@
 	)
 	(no_connect
+		(at 34.29 97.79)
+	)
+	(no_connect
 		(at 34.29 100.33)
 	)
@@
 	(wire
 		(pts
+			(xy 22.86 69.85) (xy 34.29 69.85)
+		)
+		(stroke
+			(width 0)
+			(type default)
+		)
+	)
+	(wire
+		(pts
 			(xy 180.34 17.78) (xy 193.04 17.78)
 		)
@@
 	(wire
 		(pts
-			(xy 22.86 97.79) (xy 34.29 97.79)
-		)
-		(stroke
-			(width 0)
-			(type default)
-		)
-	)
-	(wire
-		(pts
 			(xy 22.86 39.37) (xy 34.29 39.37)
 		)
@@
 		)
 	)
-	(label "P_EN"
-		(at 22.86 97.79 0)
+	(label "XOUT"
+		(at 38.1 133.35 0)
 		(fields_autoplaced yes)
 		(effects
@@
 		)
 	)
-	(label "XOUT"
-		(at 38.1 133.35 0)
+	(label "P_EN"
+		(at 22.86 69.85 0)
 		(fields_autoplaced yes)
 		(effects
