File: LogicTranslation.kicad_sch (KiCad schematic)
At the start: 31 parts, among them U11 SN74LVC1T45DCK, U12 SN74LVC1T45DCK, U2 SN74LVC1T45DCK, U3 SN74LVC1T45DCK, U4 SN74LVC1T45DCK, U5 SN74LVC1T45DCK, U6 SN74LVC1T45DCK, U7 SN74LVC1T45DCK, U8 SN74LVC1T45DCK, U9 SN74LVC1T45DCK

Commit message: update: 更新设计
Parts:
- added R24, R25, R26, R27: 22R, Resistor_SMD:R_0402_1005Metric, symbol Device:R
- added R28, R29, R30, R31, R32, R33: 100R, Resistor_SMD:R_0402_1005Metric, symbol Device:R
Connections:
- net OUT_SRST: now also R29.2; no longer U7.4 (B)
- net OUT_SWCLK/TCK: now also R24.2; no longer U2.4 (B)
- net OUT_SWDIO/TMS: now also R25.2; no longer U3.4 (B)
- net OUT_TDI: now also R27.2; no longer U5.4 (B)
- net OUT_TDO: now also R26.2; no longer U4.4 (B)
- net OUT_TRST: now also R28.2; no longer U6.4 (B)
- net OUT_UART_DTR: now also R32.2; no longer U11.4 (B)
- net OUT_UART_RTS: now also R33.2; no longer U12.4 (B)
- net OUT_UART_RX: now also R31.2; no longer U9.4 (B)
- net OUT_UART_TX: now also R30.2; no longer U8.4 (B)
- new net: R24.1, U2.4 (B)
- new net: R30.1, U8.4 (B)
- new net: R32.1, U11.4 (B)
- new net: R28.1, U6.4 (B)
- new net: R26.1, U4.4 (B)
- new net: R27.1, U5.4 (B)
- new net: R29.1, U7.4 (B)
- new net: R25.1, U3.4 (B)
- new net: R31.1, U9.4 (B)
- new net: R33.1, U12.4 (B)
